File: power.sch (KiCad schematic (older format))
At the start: 39 parts, among them P4 CONN_2, P5 KNUSB, U4 STM32F46X_LQFP176, U6 LP38691, X1 CRYSTAL

Commit message: Fix alignment of everything to 50 mil
Connections:
- wire segments 101 -> 171
Other:
- moved on the sheet: B1, C?, D1, D2, JP1, L1, P4, P5, R?, U4B, U6

Commit message: Misc. small fixes, DRC (almost) passes now.
Parts:
- removed X1: CRYSTAL, knielsenlib:2-SOJ, symbol CRYSTAL_SMD
- added X1: MA-505, symbol Crystal_Small
- gave numbers to parts that had none: 29
- renumbered U4 to U1, U6 to U3
Connections:
- wire segments 171 -> 101

Commit message: Couple small fixes and tweaks.
Some resistors added on inputs connected directly to power lines.
Few labels added.
Parts:
- added R10: 510, symbol R_Small
- added R11, R9: 10k, symbol R_Small
Connections:
- net +3V3: now also R11.1; no longer U1.171 (PDR_ON)
- net GND: now also R10.1, R9.1; no longer U1.166 (BOOT0), U1.48 (BYPASS_REG)
- net vdd12dsi: now reaches C26.1, U1.100 (Vcapdsi), U1.106 (vdd12dsi)
- new net boot0: R10.2, U1.166 (BOOT0)
- new net bypass: R9.2, U1.48 (BYPASS_REG)
- new net pdr_on: R11.2, U1.171 (PDR_ON)

Commit message: Basic netlist with footprint assignment and import into pcbnew
Parts:
- C21, C22, C25, C26: footprint (none) -> w_smd_cap:c_0805
- R10, R11, R9: footprint (none) -> w_smd_resistors:r_0805
- U1: footprint (none) -> w_smd_lqfp:LQFP-176
- X1: footprint (none) -> knielsenlib_old:2-SOJ
Changed lines of the file:
@@
 F 0 "U1" H 2500 3500 60  0000 C CNN
 F 1 "STM32F46X_LQFP176" H 2500 1975 60  0000 C CNN
-F 2 "" H 2500 3050 60  0000 C CNN
+F 2 "w_smd_lqfp:LQFP-176" H 2500 3050 60  0001 C CNN
 F 3 "" H 2500 3050 60  0000 C CNN
 	2    2500 2750
@@
 $EndComp
 Wire Wire Line
-	2100 2050 2100 2100
-Wire Wire Line
-	2100 2100 2100 2150
-Wire Wire Line
-	2100 2150 2100 2200
-Wire Wire Line
-	2100 2200 2100 2250
-Wire Wire Line
-	2100 2250 2100 2300
-Wire Wire Line
-	2100 2300 2100 2350
-Wire Wire Line
-	2100 2350 2100 2400
-Wire Wire Line
-	2100 2400 2100 2450
-Wire Wire Line
-	2100 2450 2100 2500
-Wire Wire Line
-	2100 2500 2100 2550
-Wire Wire Line
-	2100 2550 2100 2600
-Wire Wire Line
-	2100 2600 2100 2650
-Wire Wire Line
-	2100 2650 2100 2700
-Wire Wire Line
-	2100 2700 2100 2800
+	2100 2050 2100 2800
 Connection ~ 2100 2200
 Connection ~ 2100 2150
@@
 $EndComp
 Wire Wire Line
-	3225 2400 3225 2400
+	2900 2400 3225 2400
 $Comp
 L +3.3V #PWR020
@@
 	4650 2300 4650 2400
 Wire Wire Line
-	4400 2300 4550 2300
-Wire Wire Line
-	4550 2300 4650 2300
-Wire Wire Line
-	3800 3000 3800 2600
-Wire Wire Line
-	3800 2600 3800 2300
+	4400 2300 4650 2300
+Wire Wire Line
+	3800 3000 3800 2300
 Wire Wire Line
 	3800 2300 4000 2300
@@
 Connection ~ 3350 3750
 Wire Wire Line
-	3100 3750 3350 3750
-Wire Wire Line
-	3350 3750 3550 3750
+	3100 3750 3550 3750
 Wire Wire Line
 	2900 3400 3100 3400
@@
 	3100 3400 3100 3750
 Wire Wire Line
-	2900 3350 3350 3350
-Wire Wire Line
-	3350 3350 3550 3350
+	2900 3350 3550 3350
 Connection ~ 3350 3350
 Wire Wire Line
-	3750 3350 3750 3750
-Wire Wire Line
-	3750 3750 3750 3900
+	3750 3350 3750 3900
 Connection ~ 3750 3750
 Wire Wire Line
-	2900 3000 3500 3000
-Wire Wire Line
-	3500 3000 3800 3000
+	2900 3000 3800 3000
 Connection ~ 3800 2300
 Wire Wire Line
@@
 $EndComp
 Wire Wire Line
-	2925 1800 2950 1800
-Wire Wire Line
-	2950 1800 3150 1800
-Wire Wire Line
-	3150 1800 3350 1800
-Wire Wire Line
-	3350 1800 3550 1800
-Wire Wire Line
-	3550 1800 3750 1800
-Wire Wire Line
-	3750 1800 3950 1800
-Wire Wire Line
-	3950 1800 4150 1800
+	2925 1800 4150 1800
 Connection ~ 3350 1800
 $Comp
@@
 Connection ~ 6750 2550
 Wire Wire Line
-	6750 2300 6750 2550
-Wire Wire Line
-	6750 2550 6750 2600
-Wire Wire Line
-	6400 1850 6550 1850
-Wire Wire Line
-	6550 1850 6750 1850
-Wire Wire Line
-	6750 1850 7050 1850
-Wire Wire Line
-	7650 1850 7850 1850
-Wire Wire Line
-	7850 1850 8000 1850
-Wire Wire Line
-	8000 1850 8150 1850
+	6750 2300 6750 2600
+Wire Wire Line
+	6400 1850 7050 1850
+Wire Wire Line
+	7650 1850 8150 1850
 Wire Wire Line
 	6750 2000 6750 1850
@@
 Connection ~ 6550 1850
 Wire Wire Line
-	6550 2550 6750 2550
-Wire Wire Line
-	6750 2550 7050 2550
-Wire Wire Line
-	7050 2550 7850 2550
+	6550 2550 7850 2550
 Wire Wire Line
 	7850 2550 7850 2300
@@
 	7300 4950 7600 4950
 Wire Wire Line
-	8250 4950 8250 5400
-Wire Wire Line
-	8250 5400 8250 5600
+	8250 4950 8250 5600
 Wire Wire Line
 	8250 4950 8000 4950
@@
 	2650 5750 3000 5750
 Wire Wire Line
-	2650 5450 2900 5450
-Wire Wire Line
-	2900 5450 3000 5450
+	2650 5450 3000 5450
 Wire Wire Line
 	2800 6550 2800 6650
@@
 	2450 4750 2450 4800
 Wire Wire Line
-	2900 2400 3225 2400
-Wire Wire Line
-	2100 2950 2100 3000
-Wire Wire Line
-	2100 3000 2100 3050
-Wire Wire Line
-	2100 3050 2100 3100
-Wire Wire Line
-	2100 3100 2100 3150
-Wire Wire Line
-	2100 3150 2100 3200
-Wire Wire Line
-	2100 3200 2100 3250
-Wire Wire Line
-	2100 3250 2100 3300
-Wire Wire Line
-	2100 3300 2100 3350
-Wire Wire Line
-	2100 3350 2100 3400
+	2100 2950 2100 3400
 Connection ~ 2100 3000
 Connection ~ 2100 3050
@@
 Connection ~ 2100 2650
 Wire Wire Line
-	2900 2100 3025 2100
-Wire Wire Line
-	3025 2100 3100 2100
+	2900 2100 3100 2100
 Wire Wire Line
 	2900 2150 3000 2150
@@
 $EndComp
 Wire Wire Line
-	1150 1800 1350 1800
-Wire Wire Line
-	1350 1800 1550 1800
-Wire Wire Line
-	1550 1800 1750 1800
-Wire Wire Line
-	1750 1800 1950 1800
-Wire Wire Line
-	1950 1800 2150 1800
-Wire Wire Line
-	2150 1800 2350 1800
-Wire Wire Line
-	2350 1800 2550 1800
-Wire Wire Line
-	2550 1800 2750 1800
-Wire Wire Line
-	2750 1800 2950 1800
+	1150 1800 2950 1800
 Connection ~ 2150 1800
 $Comp
@@
 	3150 2650 3150 2500
 Wire Wire Line
-	2900 2500 3150 2500
-Wire Wire Line
-	3150 2500 3350 2500
+	2900 2500 3350 2500
 Connection ~ 3150 2500
 $Comp
@@
 F 0 "C26" H 3375 2550 30  0000 L CNN
 F 1 "2.2u" H 3475 2450 30  0000 L CNN
-F 2 "" H 3450 2500 60  0000 C CNN
+F 2 "w_smd_cap:c_0805" H 3450 2500 60  0001 C CNN
 F 3 "" H 3450 2500 60  0000 C CNN
 	1    3450 2500
@@
 	2950 2325 3100 2325
 Wire Wire Line
-	3100 2325 3100 2200
-Wire Wire Line
-	3100 2200 3100 2100
+	3100 2325 3100 2100
 Connection ~ 3025 2100
 Wire Wire Line
-	3100 2200 3225 2200
-Wire Wire Line
-	3225 2200 3450 2200
+	3100 2200 3450 2200
 Connection ~ 3100 2200
 $Comp
@@
 F 0 "C21" H 3235 2170 30  0000 L CNN
 F 1 "10n" H 3225 2050 30  0000 L CNN
-F 2 "" H 3225 2100 60  0000 C CNN
+F 2 "w_smd_cap:c_0805" H 3225 2100 60  0001 C CNN
 F 3 "" H 3225 2100 60  0000 C CNN
 	1    3225 2100
@@
 F 0 "C22" H 3460 2170 30  0000 L CNN
 F 1 "1u" H 3450 2050 30  0000 L CNN
-F 2 "" H 3450 2100 60  0000 C CNN
+F 2 "w_smd_cap:c_0805" H 3450 2100 60  0001 C CNN
 F 3 "" H 3450 2100 60  0000 C CNN
 	1    3450 2100
@@
 $EndComp
 Wire Wire Line
-	3225 2000 3450 2000
-Wire Wire Line
-	3450 2000 3700 2000
+	3225 2000 3700 2000
 Wire Wire Line
 	3700 2000 3700 2025
@@
 F 0 "C25" H 3635 2445 30  0000 L CNN
 F 1 "100n" H 3635 2295 30  0000 L CNN
-F 2 "" H 3625 2375 60  0000 C CNN
+F 2 "w_smd_cap:c_0805" H 3625 2375 60  0001 C CNN
 F 3 "" H 3625 2375 60  0000 C CNN
 	1    3625 2375
@@
 	3550 2500 3625 2500
 Wire Wire Line
-	3625 2475 3625 2500
-Wire Wire Line
-	3625 2500 3625 2550
+	3625 2475 3625 2550
 Connection ~ 3625 2500
 $Comp
@@
 $EndComp
 Wire Wire Line
-	1150 1600 1350 1600
-Wire Wire Line
-	1350 1600 1550 1600
-Wire Wire Line
-	1550 1600 1750 1600
-Wire Wire Line
-	1750 1600 1950 1600
-Wire Wire Line
-	1950 1600 2150 1600
-Wire Wire Line
-	2150 1600 2350 1600
-Wire Wire Line
-	2350 1600 2550 1600
-Wire Wire Line
-	2550 1600 2750 1600
-Wire Wire Line
-	2750 1600 2950 1600
-Wire Wire Line
-	2950 1600 3150 1600
-Wire Wire Line
-	3150 1600 3350 1600
-Wire Wire Line
-	3350 1600 3550 1600
-Wire Wire Line
-	3550 1600 3750 1600
-Wire Wire Line
-	3750 1600 3950 1600
-Wire Wire Line
-	3950 1600 4150 1600
-Wire Wire Line
-	4150 1600 4350 1600
+	1150 1600 4350 1600
 $Comp
 L C_Small C14
@@
 F 0 "X1" H 3350 3650 50  0000 C CNN
 F 1 "MA-505" H 3350 3450 50  0000 C CNN
-F 2 "" H 3350 3550 60  0000 C CNN
+F 2 "knielsenlib_old:2-SOJ" H 3350 3550 60  0001 C CNN
 F 3 "" H 3350 3550 60  0000 C CNN
 	1    3350 3550
@@
 F 0 "R9" V 3200 3125 30  0000 L CNN
 F 1 "10k" V 3150 3050 30  0000 L CNN
-F 2 "" H 3150 3100 60  0000 C CNN
+F 2 "w_smd_resistors:r_0805" H 3150 3100 60  0001 C CNN
 F 3 "" H 3150 3100 60  0000 C CNN
 	1    3150 3100
@@
 F 0 "R10" V 3200 3275 30  0000 L CNN
 F 1 "510" V 3150 3200 30  0000 L CNN
-F 2 "" H 3150 3250 60  0000 C CNN
+F 2 "w_smd_resistors:r_0805" H 3150 3250 60  0001 C CNN
 F 3 "" H 3150 3250 60  0000 C CNN
 	1    3150 3250
@@
 F 0 "R11" V 3575 3200 30  0000 L CNN
 F 1 "10k" V 3625 3125 30  0000 L CNN
-F 2 "" H 3625 3175 60  0000 C CNN
+F 2 "w_smd_resistors:r_0805" H 3625 3175 60  0001 C CNN
 F 3 "" H 3625 3175 60  0000 C CNN
 	1    3625 3175

Commit message: Couple small tweaks, 3d shapes.
Parts:
- X1: footprint knielsenlib_old:2-SOJ -> knielsenlib:2-SOJ
Changed lines of the file:
@@
 F 0 "X1" H 3350 3650 50  0000 C CNN
 F 1 "MA-505" H 3350 3450 50  0000 C CNN
-F 2 "knielsenlib_old:2-SOJ" H 3350 3550 60  0001 C CNN
+F 2 "knielsenlib:2-SOJ" H 3350 3550 60  0001 C CNN
 F 3 "" H 3350 3550 60  0000 C CNN
 	1    3350 3550

Commit message: Small component changes.
Fix couple of missing footprints. Make 100nF caps 0603.

Some very rough component placement to avoid overlap.
Parts:
- C10, C11, C12, C13, C14, C15, C16, C17, C18, C19, C25, C29, C5, C6, C7, C8, C9: footprint w_smd_cap:c_0805 -> w_smd_cap:c_0603
- L1: footprint SMD_Packages:SMD-0603 -> w_smd_cap:c_0603
Changed lines of the file:
@@
 F 0 "C29" H 3925 3050 30  0000 L CNN
 F 1 "100n" H 3925 2950 30  0000 L CNN
-F 2 "w_smd_cap:c_0805" H 3900 3000 60  0001 C CNN
+F 2 "w_smd_cap:c_0603" H 3900 3000 60  0001 C CNN
 F 3 "" H 3900 3000 60  0001 C CNN
 	1    3900 3000
@@
 F 0 "C15" H 3175 1750 30  0000 L CNN
 F 1 "100n" H 3175 1650 30  0000 L CNN
-F 2 "w_smd_cap:c_0805" H 3150 1700 60  0001 C CNN
+F 2 "w_smd_cap:c_0603" H 3150 1700 60  0001 C CNN
 F 3 "" H 3150 1700 60  0000 C CNN
 	1    3150 1700
@@
 F 0 "C16" H 3375 1750 30  0000 L CNN
 F 1 "100n" H 3375 1650 30  0000 L CNN
-F 2 "w_smd_cap:c_0805" H 3350 1700 60  0001 C CNN
+F 2 "w_smd_cap:c_0603" H 3350 1700 60  0001 C CNN
 F 3 "" H 3350 1700 60  0000 C CNN
 	1    3350 1700
@@
 F 0 "C17" H 3575 1750 30  0000 L CNN
 F 1 "100n" H 3575 1650 30  0000 L CNN
-F 2 "w_smd_cap:c_0805" H 3550 1700 60  0001 C CNN
+F 2 "w_smd_cap:c_0603" H 3550 1700 60  0001 C CNN
 F 3 "" H 3550 1700 60  0000 C CNN
 	1    3550 1700
@@
 F 0 "C18" H 3775 1750 30  0000 L CNN
 F 1 "100n" H 3775 1650 30  0000 L CNN
-F 2 "w_smd_cap:c_0805" H 3750 1700 60  0001 C CNN
+F 2 "w_smd_cap:c_0603" H 3750 1700 60  0001 C CNN
 F 3 "" H 3750 1700 60  0000 C CNN
 	1    3750 1700
@@
 F 0 "C19" H 3975 1750 30  0000 L CNN
 F 1 "100n" H 3975 1650 30  0000 L CNN
-F 2 "w_smd_cap:c_0805" H 3950 1700 60  0001 C CNN
+F 2 "w_smd_cap:c_0603" H 3950 1700 60  0001 C CNN
 F 3 "" H 3950 1700 60  0000 C CNN
 	1    3950 1700
@@
 F 0 "L1" V 2750 6250 40  0000 C CNN
 F 1 "30@100MHz" V 2900 6250 40  0000 C CNN
-F 2 "SMD_Packages:SMD-0603" H 2800 6250 60  0001 C CNN
+F 2 "w_smd_cap:c_0603" H 2800 6250 60  0001 C CNN
 F 3 "" H 2800 6250 60  0001 C CNN
 	1    2800 6250
@@
 F 0 "C9" H 1975 1750 30  0000 L CNN
 F 1 "100n" H 1975 1650 30  0000 L CNN
-F 2 "w_smd_cap:c_0805" H 1950 1700 60  0001 C CNN
+F 2 "w_smd_cap:c_0603" H 1950 1700 60  0001 C CNN
 F 3 "" H 1950 1700 60  0000 C CNN
 	1    1950 1700
@@
 F 0 "C10" H 2175 1750 30  0000 L CNN
 F 1 "100n" H 2175 1650 30  0000 L CNN
-F 2 "w_smd_cap:c_0805" H 2150 1700 60  0001 C CNN
+F 2 "w_smd_cap:c_0603" H 2150 1700 60  0001 C CNN
 F 3 "" H 2150 1700 60  0000 C CNN
 	1    2150 1700
@@
 F 0 "C11" H 2375 1750 30  0000 L CNN
 F 1 "100n" H 2375 1650 30  0000 L CNN
-F 2 "w_smd_cap:c_0805" H 2350 1700 60  0001 C CNN
+F 2 "w_smd_cap:c_0603" H 2350 1700 60  0001 C CNN
 F 3 "" H 2350 1700 60  0000 C CNN
 	1    2350 1700
@@
 F 0 "C12" H 2575 1750 30  0000 L CNN
 F 1 "100n" H 2575 1650 30  0000 L CNN
-F 2 "w_smd_cap:c_0805" H 2550 1700 60  0001 C CNN
+F 2 "w_smd_cap:c_0603" H 2550 1700 60  0001 C CNN
 F 3 "" H 2550 1700 60  0000 C CNN
 	1    2550 1700
@@
 F 0 "C13" H 2775 1750 30  0000 L CNN
 F 1 "100n" H 2775 1650 30  0000 L CNN
-F 2 "w_smd_cap:c_0805" H 2750 1700 60  0001 C CNN
+F 2 "w_smd_cap:c_0603" H 2750 1700 60  0001 C CNN
 F 3 "" H 2750 1700 60  0000 C CNN
 	1    2750 1700
@@
 F 0 "C8" H 1775 1750 30  0000 L CNN
 F 1 "100n" H 1775 1650 30  0000 L CNN
-F 2 "w_smd_cap:c_0805" H 1750 1700 60  0001 C CNN
+F 2 "w_smd_cap:c_0603" H 1750 1700 60  0001 C CNN
 F 3 "" H 1750 1700 60  0000 C CNN
 	1    1750 1700
@@
 F 0 "C6" H 1375 1750 30  0000 L CNN
 F 1 "100n" H 1375 1650 30  0000 L CNN
-F 2 "w_smd_cap:c_0805" H 1350 1700 60  0001 C CNN
+F 2 "w_smd_cap:c_0603" H 1350 1700 60  0001 C CNN
 F 3 "" H 1350 1700 60  0000 C CNN
 	1    1350 1700
@@
 F 0 "C7" H 1575 1750 30  0000 L CNN
 F 1 "100n" H 1575 1650 30  0000 L CNN
-F 2 "w_smd_cap:c_0805" H 1550 1700 60  0001 C CNN
+F 2 "w_smd_cap:c_0603" H 1550 1700 60  0001 C CNN
 F 3 "" H 1550 1700 60  0000 C CNN
 	1    1550 1700
@@
 F 0 "C5" H 1175 1750 30  0000 L CNN
 F 1 "100n" H 1175 1650 30  0000 L CNN
-F 2 "w_smd_cap:c_0805" H 1150 1700 60  0001 C CNN
+F 2 "w_smd_cap:c_0603" H 1150 1700 60  0001 C CNN
 F 3 "" H 1150 1700 60  0000 C CNN
 	1    1150 1700
@@
 F 0 "C25" H 3635 2445 30  0000 L CNN
 F 1 "100n" H 3635 2295 30  0000 L CNN
-F 2 "w_smd_cap:c_0805" H 3625 2375 60  0001 C CNN
+F 2 "w_smd_cap:c_0603" H 3625 2375 60  0001 C CNN
 F 3 "" H 3625 2375 60  0000 C CNN
 	1    3625 2375
@@
 F 0 "C14" H 2975 1750 30  0000 L CNN
 F 1 "100n" H 2975 1650 30  0000 L CNN
-F 2 "w_smd_cap:c_0805" H 2950 1700 60  0001 C CNN
+F 2 "w_smd_cap:c_0603" H 2950 1700 60  0001 C CNN
 F 3 "" H 2950 1700 60  0000 C CNN
 	1    2950 1700

Commit message: Fix LED polarity (+ small cleanups).
Parts:
- D1, D2: footprint w_smd_leds:Led_0805 -> LEDs:LED_0805
Changed lines of the file:
@@
 F 0 "D2" H 7800 5500 50  0000 C CNN
 F 1 "SML-211YTT86" H 7800 5300 50  0000 C CNN
-F 2 "w_smd_leds:Led_0805" H 7800 5400 60  0001 C CNN
+F 2 "LEDs:LED_0805" H 7800 5400 60  0001 C CNN
 F 3 "" H 7800 5400 60  0001 C CNN
 	1    7800 5400
@@
 F 0 "D1" H 7800 5050 50  0000 C CNN
 F 1 "SML-211UTT86" H 7800 4850 50  0000 C CNN
-F 2 "w_smd_leds:Led_0805" H 7800 4950 60  0001 C CNN
+F 2 "LEDs:LED_0805" H 7800 4950 60  0001 C CNN
 F 3 "" H 7800 4950 60  0001 C CNN
 	1    7800 4950
